Commit message: .

File: ros_arduino_bridge/urdf/new_robot_urdf.xacro (robot description, xacro)
@@ -1,164 +1,305 @@
-<?xml version="1.0" ?>
-<robot name="new_robot_urdf"
-  xmlns:xacro="http://www.ros.org/wiki/xacro">
-  <xacro:include filename="$(find ros_arduino_bridge)/urdf/materials.xacro" />
-  <xacro:include filename="$(find ros_arduino_bridge)/urdf/new_robot_urdf.trans" />
-  <xacro:include filename="$(find ros_arduino_bridge)/urdf/new_robot_urdf.gazebo" />
+<?xml version="1.0"?>
+<robot xmlns:xacro="http://www.ros.org/wiki/xacro">
+  <xacro:include filename="inertial_macros.xacro" />
+  <xacro:property name="chassis_length" value="0.290" />
+  <xacro:property name="chassis_width" value="0.170" />
+  <xacro:property name="chassis_height" value="0.036" />
+  <xacro:property name="wheel_radius" value="0.0425" />
+  <xacro:property name="wheel_thickness" value="0.038" />
+  <xacro:property name="front_wheel_offset_x" value="${0.190/2}" />
+  <xacro:property name="front_wheel_offset_y" value="${0.249/2}" />
+  <xacro:property name="front_wheel_offset_z" value="${wheel_radius}" />
+  <xacro:property name="back_wheel_offset_x" value="${0.190/2}" />
+  <xacro:property name="back_wheel_offset_y" value="${front_wheel_offset_y}" />
+  <xacro:property name="back_wheel_offset_z" value="${front_wheel_offset_z}" />
+  <xacro:property name="lidar_height" value="0.023" />
+  <xacro:property name="lidar_offset_x" value="${0.050}" />
+  <xacro:property name="lidar_offset_z" value="${chassis_height + front_wheel_offset_z}" />
+  <xacro:property name="imu_length" value="0.030" />
+  <xacro:property name="imu_width" value="0.015" />
+  <xacro:property name="imu_offset_x" value="${0.0}" />
+  <xacro:property name="imu_offset_y" value="0.0" />
+  <xacro:property name="imu_offset_z" value="${chassis_height + 0.02}" />
+  <xacro:property name="chassis_mass" value="1.0" />
+  <xacro:property name="lidar_mass" value="0.01" />
+  <xacro:property name="imu_mass" value="0.001" />
+  <xacro:property name="wheel_mass" value="0.05" />
+  <xacro:property name="mu1" value="0.25" />
+  <xacro:property name="mu2" value="0.25" />
+  <xacro:property name="sl1" value="10.0" />
+  <xacro:property name="sl2" value="10.0" />
+  <xacro:property name="centre_of_rot_offset_x" value="${-0.02}" />
+  <material name="white">
+    <color rgba="1 1 1 1" />
+  </material>
+  <material name="orange">
+    <color rgba="1 0.3 0.1 1" />
+  </material>
+  <material name="blue">
+    <color rgba="0.2 0.2 1 1" />
+  </material>
+  <material name="black">
+    <color rgba="0 0 0 1" />
+  </material>
+  <material name="red">
+    <color rgba="1 0 0 1" />
+  </material>
+  <!-- BASE LINK -->
   <link name="base_link">
-    <inertial>
-      <origin xyz="0.16003404098199894 0.07999869526838829 0.1125351775810762" rpy="0 0 0"/>
-      <mass value="42.407840579162674"/>
-      <inertia ixx="0.132584" iyy="0.40276" izz="0.45462" ixy="0.0" iyz="-3e-06" ixz="8.7e-05"/>
-    </inertial>
-    <visual>
-      <origin xyz="0 0 0" rpy="0 0 0"/>
-      <geometry>
-        <mesh filename="file://$(find ros_arduino_bridge)/meshes/base_link.stl" scale="0.001 0.001 0.001"/>
-      </geometry>
-      <material name="silver"/>
-    </visual>
-    <collision>
-      <origin xyz="0 0 0" rpy="0 0 0"/>
-      <geometry>
-        <mesh filename="file://$(find ros_arduino_bridge)/meshes/base_link.stl" scale="0.001 0.001 0.001"/>
-      </geometry>
-    </collision>
-  </link>
+  </link>
+  <!-- BASE_FOOTPRINT LINK -->
+  <joint name="base_footprint_joint" type="fixed">
+    <parent link="base_link" />
+    <child link="base_footprint" />
+    <origin xyz="0 0 0" rpy="0 0 0" />
+  </joint>
+  <link name="base_footprint">
+  </link>
+  <!-- CHASSIS LINK -->
+  <joint name="chassis_joint" type="fixed">
+    <parent link="base_link" />
+    <child link="chassis" />
+    <origin xyz="${centre_of_rot_offset_x} 0 ${-front_wheel_offset_z}" />
+  </joint>
+  <link name="chassis">
+    <visual>
+      <origin xyz="0 0 ${chassis_height/2 + front_wheel_offset_z}" />
+      <geometry>
+        <box size="${chassis_length} ${chassis_width} ${chassis_height}" />
+      </geometry>
+      <material name="orange" />
+    </visual>
+    <collision>
+      <origin xyz="0 0 ${chassis_height/2  + front_wheel_offset_z}" />
+      <geometry>
+        <box size="${chassis_length} ${chassis_width} ${chassis_height}" />
+      </geometry>
+    </collision>
+    <xacro:inertial_box mass="${chassis_mass}" x="${chassis_length}" y="${chassis_width}" z="${chassis_height}">
+      <origin xyz="0 0 ${chassis_height/2  + front_wheel_offset_z}" rpy="0 0 0" />
+    </xacro:inertial_box>
+  </link>
+  <gazebo reference="chassis">
+    <material>Gazebo/Orange</material>
+  </gazebo>
+  <joint name="front_left_wheel_joint" type="continuous">
+    <parent link="base_link" />
+    <child link="fore_left_wheel_1" />
+    <origin xyz="${front_wheel_offset_x + centre_of_rot_offset_x} ${front_wheel_offset_y} 0" rpy="-${pi/2} 0 0" />
+    <axis xyz="0 0 1" />
+  </joint>
+  <link name="fore_left_wheel_1">
+    <visual>
+      <geometry>
+        <cylinder radius="${wheel_radius}" length="${wheel_thickness}" />
+      </geometry>
+      <material name="red" />
+    </visual>
+    <collision>
+      <geometry>
+        <sphere radius="${wheel_radius}" />
+      </geometry>
+    </collision>
+    <xacro:inertial_cylinder mass="${wheel_mass}" length="${wheel_thickness}" radius="${wheel_radius}">
+      <origin xyz="0 0 0" rpy="0 0 0" />
+    </xacro:inertial_cylinder>
+  </link>
+  <gazebo reference="fore_left_wheel_1">
+    <material>Gazebo/Red</material>
+    <!-- <mu1>${mu1}</mu1>
+        <mu2>${mu2}</mu2>
+        <kp>1e5</kp>
+        <kd>1.0</kd>
+        <fdir1>1 0 0</fdir1>
+        <slip1>${sl1}</slip1>
+        <slip2>${sl2}</slip2>     -->
+  </gazebo>
+  <joint name="front_right_wheel_joint" type="continuous">
+    <parent link="base_link" />
+    <child link="fore_right_wheel_1" />
+    <origin xyz="${front_wheel_offset_x + centre_of_rot_offset_x} ${-front_wheel_offset_y} 0" rpy="${pi/2} 0 0" />
+    <axis xyz="0 0 -1" />
+  </joint>
   <link name="fore_right_wheel_1">
-    <inertial>
-      <origin xyz="1.9740023782244265e-07 -0.015499526820072326 6.938893903907228e-18" rpy="0 0 0"/>
-      <mass value="1.3808899961285064"/>
-      <inertia ixx="0.000734" iyy="0.001247" izz="0.000734" ixy="0.0" iyz="-0.0" ixz="0.0"/>
-    </inertial>
-    <visual>
-      <origin xyz="-0.256429 0.027778 -0.0425" rpy="0 0 0"/>
-      <geometry>
-        <mesh filename="file://$(find ros_arduino_bridge)/meshes/fore_right_wheel_1.stl" scale="0.001 0.001 0.001"/>
-      </geometry>
-      <material name="silver"/>
-    </visual>
-    <collision>
-      <origin xyz="-0.256429 0.027778 -0.0425" rpy="0 0 0"/>
-      <geometry>
-        <mesh filename="file://$(find ros_arduino_bridge)/meshes/fore_right_wheel_1.stl" scale="0.001 0.001 0.001"/>
-      </geometry>
-    </collision>
-  </link>
+    <visual>
+      <geometry>
+        <cylinder radius="${wheel_radius}" length="${wheel_thickness}" />
+      </geometry>
+      <material name="red" />
+    </visual>
+    <collision>
+      <geometry>
+        <sphere radius="${wheel_radius}" />
+      </geometry>
+    </collision>
+    <xacro:inertial_cylinder mass="${wheel_mass}" length="${wheel_thickness}" radius="${wheel_radius}">
+      <origin xyz="0 0 0" rpy="0 0 0" />
+    </xacro:inertial_cylinder>
+  </link>
+  <gazebo reference="fore_right_wheel_1">
+    <material>Gazebo/Red</material>
+    <!-- <mu1>${mu1}</mu1>
+        <mu2>${mu2}</mu2>
+        <kp>1e5</kp>
+        <kd>1.0</kd>
+        <fdir1>1 0 0</fdir1>
+        <slip1>${sl1}</slip1>
+        <slip2>${sl2}</slip2>     -->
+  </gazebo>
+  <joint name="back_left_wheel_joint" type="continuous">
+    <parent link="base_link" />
+    <child link="back_left_wheel_1" />
+    <origin xyz="${-back_wheel_offset_x + centre_of_rot_offset_x} ${back_wheel_offset_y} 0" rpy="-${pi/2} 0 0" />
+    <axis xyz="0 0 1" />
+  </joint>
+  <link name="back_left_wheel_1">
+    <visual>
+      <geometry>
+        <cylinder radius="${wheel_radius}" length="${wheel_thickness}" />
+      </geometry>
+      <material name="blue" />
+    </visual>
+    <collision>
+      <geometry>
+        <sphere radius="${wheel_radius}" />
+      </geometry>
+    </collision>
+    <xacro:inertial_cylinder mass="${wheel_mass}" length="${wheel_thickness}" radius="${wheel_radius}">
+      <origin xyz="0 0 0" rpy="0 0 0" />
+    </xacro:inertial_cylinder>
+  </link>
+  <gazebo reference="back_left_wheel_1">
+    <material>Gazebo/Blue</material>
+    <!-- <mu1>${mu1}</mu1>
+        <mu2>${mu2}</mu2>
+        <kp>1e5</kp>
+        <kd>1.0</kd>
+        <fdir1>1 0 0</fdir1>
+        <slip1>${sl1}</slip1>
+        <slip2>${sl2}</slip2>     -->
+  </gazebo>
+  <joint name="back_right_wheel_joint" type="continuous">
+    <parent link="base_link" />
+    <child link="back_right_wheel_1" />
+    <origin xyz="${-back_wheel_offset_x + centre_of_rot_offset_x} ${-back_wheel_offset_y} 0" rpy="${pi/2} 0 0" />
+    <axis xyz="0 0 -1" />
+  </joint>
   <link name="back_right_wheel_1">
-    <inertial>
-      <origin xyz="1.9740023783632044e-07 -0.015499526820072333 0.0" rpy="0 0 0"/>
-      <mass value="1.3808899961285064"/>
-      <inertia ixx="0.000734" iyy="0.001247" izz="0.000734" ixy="0.0" iyz="0.0" ixz="0.0"/>
-    </inertial>
-    <visual>
-      <origin xyz="-0.066429 0.027778 -0.0425" rpy="0 0 0"/>
-      <geometry>
-        <mesh filename="file://$(find ros_arduino_bridge)/meshes/back_right_wheel_1.stl" scale="0.001 0.001 0.001"/>
-      </geometry>
-      <material name="silver"/>
-    </visual>
-    <collision>
-      <origin xyz="-0.066429 0.027778 -0.0425" rpy="0 0 0"/>
-      <geometry>
-        <mesh filename="file://$(find ros_arduino_bridge)/meshes/back_right_wheel_1.stl" scale="0.001 0.001 0.001"/>
-      </geometry>
-    </collision>
-  </link>
-  <link name="fore_left_wheel_1">
-    <inertial>
-      <origin xyz="1.9740023782244265e-07 0.015499969520726242 0.0" rpy="0 0 0"/>
-      <mass value="1.3808899961285064"/>
-      <inertia ixx="0.000734" iyy="0.001247" izz="0.000734" ixy="0.0" iyz="-0.0" ixz="0.0"/>
-    </inertial>
-    <visual>
-      <origin xyz="-0.256429 -0.187668 -0.0425" rpy="0 0 0"/>
-      <geometry>
-        <mesh filename="file://$(find ros_arduino_bridge)/meshes/fore_left_wheel_1.stl" scale="0.001 0.001 0.001"/>
-      </geometry>
-      <material name="silver"/>
-    </visual>
-    <collision>
-      <origin xyz="-0.256429 -0.187668 -0.0425" rpy="0 0 0"/>
-      <geometry>
-        <mesh filename="file://$(find ros_arduino_bridge)/meshes/fore_left_wheel_1.stl" scale="0.001 0.001 0.001"/>
-      </geometry>
-    </collision>
-  </link>
-  <link name="back_left_wheel_1">
-    <inertial>
-      <origin xyz="1.97400237864076e-07 0.015499969520726242 0.0" rpy="0 0 0"/>
-      <mass value="1.3808899961285062"/>
-      <inertia ixx="0.000734" iyy="0.001247" izz="0.000734" ixy="0.0" iyz="-0.0" ixz="0.0"/>
-    </inertial>
-    <visual>
-      <origin xyz="-0.066429 -0.187668 -0.0425" rpy="0 0 0"/>
-      <geometry>
-        <mesh filename="file://$(find ros_arduino_bridge)/meshes/back_left_wheel_1.stl" scale="0.001 0.001 0.001"/>
-      </geometry>
-      <material name="silver"/>
-    </visual>
-    <collision>
-      <origin xyz="-0.066429 -0.187668 -0.0425" rpy="0 0 0"/>
-      <geometry>
-        <mesh filename="file://$(find ros_arduino_bridge)/meshes/back_left_wheel_1.stl" scale="0.001 0.001 0.001"/>
-      </geometry>
-    </collision>
-  </link>
-  <link name="lidar_1">
-    <inertial>
-      <origin xyz="-2.7755575615628914e-17 0.0 0.012249999999999955" rpy="0 0 0"/>
-      <mass value="0.7285890320350371"/>
-      <inertia ixx="0.000256" iyy="0.000256" izz="0.000439" ixy="-0.0" iyz="0.0" ixz="0.0"/>
-    </inertial>
-    <visual>
-      <origin xyz="-0.16 -0.08 -0.1655" rpy="0 0 0"/>
-      <geometry>
-        <mesh filename="file://$(find ros_arduino_bridge)/meshes/lidar_1.stl" scale="0.001 0.001 0.001"/>
-      </geometry>
-      <material name="silver"/>
-    </visual>
-    <collision>
-      <origin xyz="-0.16 -0.08 -0.1655" rpy="0 0 0"/>
-      <geometry>
-        <mesh filename="file://$(find ros_arduino_bridge)/meshes/lidar_1.stl" scale="0.001 0.001 0.001"/>
-      </geometry>
-    </collision>
-  </link>
-  <joint name="front_right_wheel_joint" type="continuous">
-    <origin xyz="0.256429 -0.027778 0.0425" rpy="0 0 0"/>
-    <parent link="base_link"/>
-    <child link="fore_right_wheel_1"/>
-    <axis xyz="0.0 -1.0 0.0"/>
-  </joint>
-  <joint name="back_right_wheel_joint" type="continuous">
-    <origin xyz="0.066429 -0.027778 0.0425" rpy="0 0 0"/>
-    <parent link="base_link"/>
-    <child link="back_right_wheel_1"/>
-    <axis xyz="0.0 -1.0 0.0"/>
-  </joint>
-  <joint name="front_left_wheel_joint" type="continuous">
-    <origin xyz="0.256429 0.187668 0.0425" rpy="0 0 0"/>
-    <parent link="base_link"/>
-    <child link="fore_left_wheel_1"/>
-    <axis xyz="0.0 1.0 0.0"/>
-  </joint>
-  <joint name="back_left_wheel_joint" type="continuous">
-    <origin xyz="0.066429 0.187668 0.0425" rpy="0 0 0"/>
-    <parent link="base_link"/>
-    <child link="back_left_wheel_1"/>
-    <axis xyz="0.0 1.0 0.0"/>
-  </joint>
-  <joint name="lidar_joint" type="fixed">
-    <origin xyz="0.16 0.08 0.1655" rpy="0 0 0"/>
-    <parent link="base_link"/>
-    <child link="lidar_1"/>
-  </joint>
-  <!-- Add laser frame for SLAM -->
+    <visual>
+      <geometry>
+        <cylinder radius="${wheel_radius}" length="${wheel_thickness}" />
+      </geometry>
+      <material name="blue" />
+    </visual>
+    <collision>
+      <geometry>
+        <sphere radius="${wheel_radius}" />
+      </geometry>
+    </collision>
+    <xacro:inertial_cylinder mass="${wheel_mass}" length="${wheel_thickness}" radius="${wheel_radius}">
+      <origin xyz="0 0 0" rpy="0 0 0" />
+    </xacro:inertial_cylinder>
+  </link>
+  <gazebo reference="back_right_wheel_1">
+    <material>Gazebo/Blue</material>
+    <!-- <mu1>${mu1}</mu1>
+        <mu2>${mu2}</mu2>
+        <kp>1e5</kp>
+        <kd>1.0</kd>
+        <fdir1>1 0 0</fdir1>
+        <slip1>${sl1}</slip1>
+        <slip2>${sl2}</slip2>     -->
+  </gazebo>
+  <joint name="laser_joint" type="fixed">
+    <parent link="chassis" />
+    <child link="laser" />
+    <origin xyz="${lidar_offset_x} 0 ${lidar_offset_z + 0.05}" rpy="0 0 0" />
+  </joint>
   <link name="laser">
-  </link>
-  <joint name="laser_joint" type="fixed">
-    <origin xyz="0.0 0.0 0.012" rpy="0 0 0"/>
-    <parent link="lidar_1"/>
-    <child link="laser"/>
-  </joint>
+    <visual>
+      <geometry>
+        <cylinder radius="0.05" length="${lidar_height}" />
+      </geometry>
+      <material name="white" />
+    </visual>
+    <visual>
+      <origin xyz="0 0 -0.05" />
+      <geometry>
+        <cylinder radius="0.01" length="0.1" />
+      </geometry>
+      <material name="white" />
+    </visual>
+    <collision>
+      <geometry>
+        <cylinder radius="0.05" length="${lidar_height}" />
+      </geometry>
+    </collision>
+    <xacro:inertial_cylinder mass="${lidar_mass}" length="0.04" radius="0.05">
+      <origin xyz="0 0 0" rpy="0 0 0" />
+    </xacro:inertial_cylinder>
+  </link>
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
Commit message: Meshes with IMU link

File: ros_arduino_bridge/urdf/new_robot_urdf.xacro (robot description, xacro)
@@ -162,3 +162,30 @@
     <child link="laser"/>
   </joint>
+  <!-- IMU Link (MPU6050) - 3cm below base_link center -->
+  <link name="imu_link">
+    <inertial>
+      <origin xyz="0 0 0" rpy="0 0 0"/>
+      <mass value="0.005"/>  <!-- MPU6050 is ~5 grams -->
+      <inertia ixx="0.000001" iyy="0.000001" izz="0.000001"
+               ixy="0.0" iyz="0.0" ixz="0.0"/>
+    </inertial>
+    <visual>
+      <origin xyz="-0.16 -0.08 0.03" rpy="0 0 0"/>
+      <geometry>
+        <mesh filename="file://$(find ros_arduino_bridge)/meshes/imu_1.stl" scale="0.001 0.001 0.001"/>
+      </geometry>
+      <material name="silver"/>
+    </visual>
+    <collision>
+      <origin xyz="-0.16 -0.08 0.03" rpy="0 0 0"/>
+      <geometry>
+        <mesh filename="file://$(find ros_arduino_bridge)/meshes/imu_1.stl" scale="0.001 0.001 0.001"/>
+      </geometry>
+    </collision>
+  </link>
+  <joint name="imu_joint" type="fixed">
+    <origin xyz="0.0 0.0 -0.03" rpy="0 0 0"/>
+    <parent link="base_link"/>
+    <child link="imu_link"/>
+  </joint>
 </robot>

Commit message: Fixes

File: ros_arduino_bridge/urdf/new_robot_urdf.xacro (robot description, xacro)
@@ -165,11 +165,10 @@
   <link name="imu_link">
     <inertial>
-      <origin xyz="0 0 0" rpy="0 0 0"/>
-      <mass value="0.005"/>  <!-- MPU6050 is ~5 grams -->
-      <inertia ixx="0.000001" iyy="0.000001" izz="0.000001"
-               ixy="0.0" iyz="0.0" ixz="0.0"/>
+      <origin xyz="1.974002378779538e-07 0.0 -0.000999999999999987" rpy="0 0 0"/>
+      <mass value="0.15700000000000014"/>
+      <inertia ixx="0.000131" iyy="0.000131" izz="0.000262" ixy="0.0" iyz="0.0" ixz="0.0"/>
     </inertial>
     <visual>
-      <origin xyz="-0.16 -0.08 0.03" rpy="0 0 0"/>
+      <origin xyz="-0.161429 -0.08 -0.0625" rpy="0 0 0"/>
       <geometry>
         <mesh filename="file://$(find ros_arduino_bridge)/meshes/imu_1.stl" scale="0.001 0.001 0.001"/>
@@ -178,5 +177,5 @@
     </visual>
     <collision>
-      <origin xyz="-0.16 -0.08 0.03" rpy="0 0 0"/>
+      <origin xyz="-0.161429 -0.08 -0.0625" rpy="0 0 0"/>
       <geometry>
         <mesh filename="file://$(find ros_arduino_bridge)/meshes/imu_1.stl" scale="0.001 0.001 0.001"/>
@@ -185,5 +184,5 @@
   </link>
   <joint name="imu_joint" type="fixed">
-    <origin xyz="0.0 0.0 -0.03" rpy="0 0 0"/>
+    <origin xyz="0.161429 0.08 0.0625" rpy="0 0 0"/>
     <parent link="base_link"/>
     <child link="imu_link"/>
